Commit message: full bender urdf

File: src/src/bender_5_urdf/src/bender_5.urdf (robot description, URDF)
Before this commit: robot waveshare, 2 links, 1 joints
Links:
- added link synexens_link; visual box size=0.1 0.1 0.1
- added link vectornav_link; visual box size=0.1 0.1 0.1
- added link vive_link; visual box size=0.1 0.1 0.1
Joints:
- added joint synexens_joint: type fixed, parent base_link, child synexens_link, origin xyz=${synexens_xoff} ${-synexens_yoff} ${synexens_height-chassis_zoff} rpy=0 0 0, axis 0 1 0
- added joint vectornav_link: type fixed, parent base_link, child vectornav_link, origin xyz=0.0 0.0 0.0 rpy=0 0 0, axis 0 1 0
- added joint vive_joint: type fixed, parent base_link, child vive_link, origin xyz=${-vive_xoff} ${vive_yoff} ${chassis_height/2.0} rpy=0 0 0, axis 0 1 0

Commit message: update parameters

File: src/src/bender_5_urdf/src/bender_5.urdf (robot description, URDF)
Before this commit: robot waveshare, 5 links, 4 joints
Joints:
- joint synexens_joint: origin xyz=${synexens_xoff} ${-synexens_yoff} ${synexens_height-chassis_zoff} rpy=0 0 0 -> xyz=${synexens_xoff} ${-synexens_yoff} ${synexens_height-chassis_zoff} rpy=-1.63 0 ${-pi/2}

Commit message: fixes

File: src/src/bender_5_urdf/src/bender_5.urdf (robot description, URDF)
Before this commit: robot waveshare, 5 links, 4 joints
Joints:
- joint vive_joint: origin xyz=${-vive_xoff} ${vive_yoff} ${chassis_height/2.0} rpy=0 0 0 -> xyz=${-vive_xoff} ${vive_yoff} ${chassis_height/2.0} rpy=0 0 ${-pi/2}

Commit message: launch file updates

File: src/src/bender_5_urdf/src/bender_5.urdf (robot description, URDF)
Before this commit: robot waveshare, 5 links, 4 joints
Joints:
- joint vive_joint: origin xyz=${-vive_xoff} ${vive_yoff} ${chassis_height/2.0} rpy=0 0 ${-pi/2} -> xyz=${-vive_xoff} ${vive_yoff} ${(chassis_height/2.0)+0.05} rpy=0 0 ${-pi/2}

Commit message: update param files

File: src/src/bender_5_urdf/src/bender_5.urdf (robot description, URDF)
Before this commit: robot waveshare, 5 links, 4 joints
Joints:
- joint vive_joint: origin xyz=${-vive_xoff} ${vive_yoff} ${(chassis_height/2.0)+0.05} rpy=0 0 ${-pi/2} -> xyz=${-vive_xoff} ${vive_yoff} ${(chassis_height/2.0)+0.10} rpy=0 0 ${-pi/2}
